File: pcb/smt32triple/control.kicad_pcb (KiCad board)
At the start: 2 copper layers, 60 x 41 mm, 43 parts, among them J1 USB_C_Receptacle_USB2.0, J4 Term, J5 Term, J6 Term, P1 ST-Link, P2 ST-Link, P3 UG-2864ASWPG01, P4 har-flexicon 2,54 MSH-4, P5 har-flexicon 2,54 MSH-4, P6 har-flexicon 2,54 MSH-4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

Commit message: Cleanup, add casing
Parts:
- added C15: 100n, Capacitor_SMD:C_0603_1608Metric, F.Cu at (113.3, 105.9)
- added JP3: Jumper_2_Open, local:Jumper, B.Cu at (89.5, 106.0)
- added JP4: Jumper_2_Open, local:Jumper, B.Cu at (110.4, 106.0)
- added R10: 33k, Resistor_SMD:R_0603_1608Metric, F.Cu at (85.7, 155.1)
- added R5: 120k, Resistor_SMD:R_0603_1608Metric, F.Cu at (85.7, 142.6)
- added R6: 33k, Resistor_SMD:R_0603_1608Metric, F.Cu at (85.7, 145.1)
- added R7: 120k, Resistor_SMD:R_0603_1608Metric, F.Cu at (85.7, 147.6)
- added R8: 33k, Resistor_SMD:R_0603_1608Metric, F.Cu at (85.7, 150.1)
- added R9: 120k, Resistor_SMD:R_0603_1608Metric, F.Cu at (85.7, 152.6)
- moved C13 18.1 mm to (70.2, 107.5), turned to 90 degrees
- moved C14 16.5 mm to (91.8, 107.7), turned to 180 degrees
- moved D5 15.2 mm to (83.8, 110.2)
- moved J5 13.9 mm to (88.7, 104.8)
- moved U5 6.89 mm to (87.8, 110.2)
- moved D6 3.85 mm to (118.2, 110.2)
- moved C1 3.63 mm to (74.7, 130.7)
- moved C2 3.63 mm to (74.0, 136.2)
- moved JP1 3.63 mm to (71.8, 131.0)
- moved R1 3.63 mm to (76.7, 135.6)
- moved R2 3.63 mm to (76.7, 133.1)
- moved U2 3.63 mm to (74.2, 133.5)
- moved D4 3.61 mm to (77.4, 110.2)
- moved P3 3.50 mm to (100.0, 111.5)
- moved P4 3.35 mm to (77.0, 102.1)
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- renumbered R4 to R1, R5 to R2, R1 to R3, R2 to R4
Connections:
- U1 pad 10: DISP_nRST -> unconnected-(U1-PA2-Pad10)
- U1 pad 30: SW -> unconnected-(U1-PA8-Pad30)
- U1 pad 4: SW -> DISP_nRST
- U1 pad 46: unconnected-(U1-PB8-Pad46) -> SW
- U4 pad 2: +3V3 -> GND
- U5 pad 2: +3V3 -> GND
- U6 pad 2: +3V3 -> GND
Routing:
- net Net-(D5-A): track 20.2 -> 50.7 mm, vias 1 -> 2
- net SW: track 45.7 -> 19.8 mm
- net GND: track 325.3 -> 301.0 mm, vias 22 -> 23
- net +15V: track 82.4 -> 95.7 mm
- net RS485_2_A: track 5.60 -> 17.3 mm
- net RS485_2_B: track 5.72 -> 16.4 mm
- net Net-(D6-A): track 19.9 -> 27.9 mm, vias 1 -> 2
- net Net-(J5-Pin_a2): track 12.1 -> 5.49 mm
- net Net-(J5-Pin_a1): track 8.56 -> 2.31 mm
- net Net-(D4-A): track 20.4 -> 26.6 mm, vias 1 -> 2
- net RS485_2_TX: track 34.8 -> 29.2 mm
- net DISP_nRST: track 7.98 -> 13.5 mm, vias 0 -> 2
- net RS485_2_DE: track 20.8 -> 15.6 mm
- net DISP_SCK: track 11.2 -> 14.7 mm
- net DISP_MOSI: track 15.0 -> 18.5 mm
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Other:
- board size 60 x 41 mm -> 62 x 39.5 mm
