File: pcb/smt32triple/control.kicad_sch (KiCad schematic)
At the start: 25 parts, among them J1 USB_C_Receptacle_USB2.0, P1 ST-Link, P2 ST-Link, P3 UG-2864ASWPG01, SW1 RotaryEncoder_Switch, U1 STM32G431CBUx, U3 BME680, U7 TPS82130

Commit message: Cleanup, add casing
Connections:
- net DISP_nRST: now also U1.4 (PC15); no longer U1.10 (PA2)
- net SW: now also U1.46 (PB8); no longer U1.30 (PA8), U1.4 (PC15)
Other:
- note added: "3x RS485 / LED Strip"
- note added: "SPI1"
- note removed: "3x LED Strip"
- moved on the sheet: C3, R10, U1
