File: pcb/smt32triple/interface.kicad_sch (KiCad schematic)
At the start: 17 parts, among them J2 Term, P1 har-flexicon 2,54 MSH-4, P2 WAGO2061-602, U3 SP3485CN

Commit message: Cleanup, add casing
Parts:
- added C3: 100n, Capacitor_SMD:C_0603_1608Metric, symbol Device:C
- added JP3, JP4: Jumper_2_Open, local:Jumper, symbol Jumper:Jumper_2_Open
- added R10 (x3): 33k, Resistor_SMD:R_0603_1608Metric, symbol Device:R
- added R10 (x3): 120k, Resistor_SMD:R_0603_1608Metric, symbol Device:R
Connections:
- net +15V: now also R10.1, R10.1, R10.1
- net +3V3: now also C3.1; no longer U3.2 (~{RE}), U3.2 (~{RE}), U3.2 (~{RE})
- net GND: now also U3.2 (~{RE}), U3.2 (~{RE}), U3.2 (~{RE}), C3.2, R10.2, R10.2, R10.2
- net at D2.2 (A), P1.2 (Pin_2), P2.2 (Pin_2): now also JP3.2 (B), JP4.1 (A)
- net at D2.2 (A), P1.2 (Pin_2), P2.2 (Pin_2): now also JP4.2 (B)
- net at D2.2 (A), P1.2 (Pin_2), P2.2 (Pin_2): now also JP3.1 (A)
- new net: R10.1, R10.2 (x3)
Other:
- note added: "LED Strip 1"
- note added: "LED Strip 2"
- note added: "LED Strip 3"
- note removed: "LED Strip"
