File: pcb/g431Triple/control.kicad_sch (KiCad schematic)
At the start: 34 parts, among them J1 TYPE-C 16PIN 2MD(073), P1 FTSH-107-01-L-DV-K, P2 ST-Link, P3 AFC07-S24FCC-00, SW1 RotaryEncoder_Switch, U1 STM32G431CBUx, U2 TPS82130, U3 BME680, U7 TSOP38338, X1 O24.000000-JSO21C1LC-D-3.3-T3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

Commit message: Works on g431Triple
Parts:
- C5: renamed from C2; symbol Device:C -> Device:C_Small
- renumbered C2 to C10, C2 to C11, C2 to C13, C2 to C14, C1 to C3, C2 to C4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
Other:
- moved on the sheet: C5, C6
